Commit message: saved config for the localization

File: sensor_kit/mach_e_sensor_kit_launch/mach_e_sensor_kit_description/urdf/sensor_kit.xacro (robot description, xacro)
@@ -44,7 +44,6 @@
       fps="100"
     />
-  </xacro:macro>
-      <!-- imu -->
-    <!-- <xacro:imu_macro
+          <!-- imu -->
+    <xacro:imu_macro
       name="imu"
       parent="sensor_kit_base_link"
@@ -57,4 +56,5 @@
       yaw="${calibration['sensor_kit_base_link']['imu_link']['yaw']}"
       fps="100"
-    /> -->
+    />
+  </xacro:macro>
 </robot>
