Commit message: Switch sensing to LUCID camera0 with camera-lidar fusion and mach-e calibration
Replace the v4l2 traffic-light camera with the LUCID arena camera (camera0)
in common_sensor_launch, default perception_mode to camera_lidar_fusion,
point traffic light recognition at camera0, and add a launch_dummy_perception
option. Update sensor_kit_calibration for the actual mounting positions,
raise max_vel to 20 m/s, and fix the Ouster IP comments to valid YAML.

Co-Authored-By: Claude Fable 5.1 <noreply@anthropic.com>

File: sensor_kit/mach_e_sensor_kit_launch/mach_e_sensor_kit_description/sensor/camera/urdf/monocular_camera.xacro (robot description, xacro)
@@ -1,24 +1,28 @@
 <?xml version="1.0"?>
 <robot xmlns:xacro="http://ros.org/wiki/xacro">
-  <xacro:macro name="monocular_camera_macro" params="name parent namespace x y z roll pitch yaw fps width height fov">
+  <xacro:macro name="monocular_camera_macro"
+               params="name parent namespace x y z roll pitch yaw fps width height fov">
     <xacro:property name="sensor_box" value="0.05"/>
     <xacro:property name="mass" value="0.1"/>
+    <!-- camera link -->
     <joint name="${name}_joint" type="fixed">
-      <origin rpy="${roll} ${pitch} ${yaw}" xyz="${x} ${y} ${z}"/>
+      <origin
+        xyz="${x} ${y} ${z}"
+        rpy="${roll} ${pitch} ${yaw}"/>
       <parent link="${parent}"/>
-      <child link="${name}_link"/>
+      <child link="${name}/camera_link"/>
     </joint>
-    <link name="${name}_link">
+    <link name="${name}/camera_link">
       <visual>
         <geometry>
           <box size="${sensor_box} ${sensor_box} ${sensor_box}"/>
         </geometry>
-        <origin rpy="0 0 0" xyz="0 0 0"/>
+        <origin xyz="0 0 0" rpy="0 0 0"/>
         <material name="red">
-          <color rgba="1.0 0.0 0.0 1.0"/>
+          <color rgba="1 0 0 1"/>
         </material>
       </visual>
       <inertial>
-        <origin rpy="0 0 0" xyz="0 0 0"/>
+        <origin xyz="0 0 0" rpy="0 0 0"/>
         <mass value="${mass}"/>
         <inertia
@@ -28,9 +32,8 @@
           iyy="${(sensor_box*sensor_box+sensor_box*sensor_box)*mass/12.0}"
           iyz="0.0"
-          izz="${(sensor_box*sensor_box+sensor_box*sensor_box)*mass/12.0}"
-        />
+          izz="${(sensor_box*sensor_box+sensor_box*sensor_box)*mass/12.0}"/>
       </inertial>
       <collision>
-        <origin rpy="0 0 0" xyz="0 0 0"/>
+        <origin xyz="0 0 0" rpy="0 0 0"/>
         <geometry>
           <box size="${sensor_box} ${sensor_box} ${sensor_box}"/>
@@ -38,51 +41,14 @@
       </collision>
     </link>
+    <!-- optical link, REP-103 optical convention (x right, y down, z forward).
+         Image/CameraInfo headers must carry this frame rather than the body link,
+         because the projection nodes treat the header frame z axis as depth.
+         Keep colons out of these comments, the URDF is YAML-parsed as a parameter. -->
     <joint name="${name}_optical_joint" type="fixed">
-      <origin rpy="${-pi/2} 0 ${-pi/2}" xyz="0 0 0"/>
-      <parent link="${name}_link"/>
-      <child link="${name}_optical_link"/>
+      <origin xyz="0 0 0" rpy="${-pi/2} 0 ${-pi/2}"/>
+      <parent link="${name}/camera_link"/>
+      <child link="${name}/camera_optical_link"/>
     </joint>
-    <link name="${name}_optical_link"/>
-    <!-- camera -->
-    <gazebo reference="${name}_link">
-      <material>Gazebo/Black</material>
-      <sensor type="camera" name="${name}">
-        <update_rate>${fps}</update_rate>
-        <camera name="${name}">
-          <horizontal_fov>${fov}</horizontal_fov>
-          <image>
-            <width>${width}</width>
-            <height>${height}</height>
-            <format>R8G8B8</format>
-          </image>
-          <clip>
-            <near>0.02</near>
-            <far>300</far>
-          </clip>
-          <noise>
-            <type>gaussian</type>
-            <!-- Noise is sampled independently per pixel on each frame.
-                 That pixel's noise value is added to each of its color
-                 channels, which at that point lie in the range [0,1]. -->
-            <mean>0.0</mean>
-            <stddev>0.007</stddev>
-          </noise>
-        </camera>
-        <plugin name="camera_controller" filename="libgazebo_ros_camera.so">
-          <alwaysOn>true</alwaysOn>
-          <updateRate>0.0</updateRate>
-          <cameraName>${namespace}</cameraName>
-          <imageTopicName>image_raw</imageTopicName>
-          <cameraInfoTopicName>camera_info</cameraInfoTopicName>
-          <frameName>${name}_optical_link</frameName>
-          <hackBaseline>0.0</hackBaseline>
-          <distortionK1>0.0</distortionK1>
-          <distortionK2>0.0</distortionK2>
-          <distortionK3>0.0</distortionK3>
-          <distortionT1>0.0</distortionT1>
-          <distortionT2>0.0</distortionT2>
-        </plugin>
-      </sensor>
-    </gazebo>
+    <link name="${name}/camera_optical_link"/>
   </xacro:macro>
 </robot>

File: sensor_kit/mach_e_sensor_kit_launch/mach_e_sensor_kit_description/urdf/sensor_kit.xacro (robot description, xacro)
@@ -57,4 +57,20 @@
       fps="100"
     />
+    <!-- camera disabled for lidar-only bringup. Re-enable by removing this comment wrapper. -->
+<xacro:monocular_camera_macro
+      name="camera_top"
+      parent="${sensor_kit_base_link}"
+      namespace="camera_top"
+      x="${calibration['sensor_kit_base_link']['camera_top/camera_link']['x']}"
+      y="${calibration['sensor_kit_base_link']['camera_top/camera_link']['y']}"
+      z="${calibration['sensor_kit_base_link']['camera_top/camera_link']['z']}"
+      roll="${calibration['sensor_kit_base_link']['camera_top/camera_link']['roll']}"
+      pitch="${calibration['sensor_kit_base_link']['camera_top/camera_link']['pitch']}"
+      yaw="${calibration['sensor_kit_base_link']['camera_top/camera_link']['yaw']}"
+      fps="30"
+      width="1920"
+      height="1080"
+      fov="1.5708"
+    />
   </xacro:macro>
 </robot>
